File: elec/Control Board/Control_1v1/Control_1v1/Adafruit-MAX31850-thermocouple-breakout-board.kicad_sch (KiCad schematic)
At the start: 37 parts, among them J11 Screw_Terminal_01x02, J2 MAX31850K

Commit message: Update schematic to reflect some reworks to V1.1 assemblies. 5V to Display. Display signal names. J35 pin8 to 10 short.
Other:
- title: Control Interconnect Board OEDCS -> Control Interconnect Board OEDCS With Reworks
Changed lines of the file:
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@@
   (paper "USLedger")
   (title_block
-    (title "Control Interconnect Board OEDCS")
-    (date "2023-10-10")
+    (title "Control Interconnect Board OEDCS With Reworks")
+    (date "2023-12-06")
     (rev "Rev 1.1")
     (company "Public Invention")
