File: elec/Control Board/Control_1v1/Control_1v1/BreadBoard30P.kicad_sch (KiCad schematic)
At the start: 22 parts, among them J1 Conn_02x06_Odd_Even, J10 Conn_01x30, J11 Conn_01x30, J12 Conn_01x30, J13 Conn_01x30, J14 Conn_01x30, J15 Conn_01x30, J16 Conn_01x30, J17 Conn_01x30, J18 Conn_02x06_Odd_Even, J19 Conn_02x06_Odd_Even, J2 Conn_02x06_Odd_Even, J20 Conn_02x06_Odd_Even, J21 Conn_02x06_Odd_Even, J22 Conn_02x06_Odd_Even, J3 Conn_02x06_Odd_Even, J4 Conn_02x06_Odd_Even, J5 Conn_02x06_Odd_Even, J6 Conn_01x30, J7 Conn_01x30, J8 Conn_01x30, J9 Conn_01x30

Commit message: Update schematic to reflect some reworks to V1.1 assemblies. 5V to Display. Display signal names. J35 pin8 to 10 short.
Other:
- title: Control Interconnect Board OEDCS -> Control Interconnect Board OEDCS With Reworks
Changed lines of the file:
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@@
   (paper "USLetter")
   (title_block
-    (title "Control Interconnect Board OEDCS")
-    (date "2023-10-10")
+    (title "Control Interconnect Board OEDCS With Reworks")
+    (date "2023-12-06")
     (rev "Rev 1.1")
     (company "Public Invention")
