File: elec/Control Board/Control_1v1/Control_1v1/Fan controller.kicad_sch (KiCad schematic)
At the start: 37 parts, among them J10 Conn_01x05, J11 Conn_01x04, J12 Conn_01x07, J20 Conn_01x04, J6 DB25_Female_MountingHoles, J9 Conn_01x04, Q2 NCE01P30K, Q601 BSS138

Commit message: Update schematic to reflect some reworks to V1.1 assemblies. 5V to Display. Display signal names. J35 pin8 to 10 short.
Other:
- title: Control Interconnect Board OEDCS -> Control Interconnect Board OEDCS With Reworks
Changed lines of the file:
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@@
   (paper "USLedger")
   (title_block
-    (title "Control Interconnect Board OEDCS")
-    (date "2023-10-10")
+    (title "Control Interconnect Board OEDCS With Reworks")
+    (date "2023-12-06")
     (rev "Rev 1.1")
     (company "Public Invention")

Commit message: Find part for D1 and D2 footprint compatible 83
Parts:
- D1, D2: Distributor 1 PN C841097 -> C2857227
Changed lines of the file:
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@@
       (effects (font (size 1.27 1.27)) hide)
     )
-    (property "Datasheet" "https://assets.nexperia.com/documents/data-sheet/BZV55_SER.pdf  BZV55B3V3" (at 250.19 91.44 0)
+    (property "Datasheet" "https://assets.nexperia.com/documents/data-sheet/BZV55_SER.pdf  BZV55B3V3,  ZMM5231.pdf" (at 250.19 91.44 0)
       (effects (font (size 1.27 1.27)) hide)
     )
@@
       (effects (font (size 1.27 1.27)) hide)
     )
-    (property "Distributor 1 PN" "C841097" (at 250.19 91.44 0)
+    (property "Distributor 1 PN" "C2857227" (at 250.19 91.44 0)
       (effects (font (size 1.27 1.27)) hide)
     )
@@
       (effects (font (size 1.27 1.27)) hide)
     )
-    (property "Distributor 1 PN" "C841097" (at 265.43 144.78 0)
+    (property "Distributor 1 PN" "C2857227" (at 265.43 144.78 0)
       (effects (font (size 1.27 1.27)) hide)
     )
