File: elec/Control Board/Control_1v2/SSR Interface.kicad_sch (KiCad schematic)
At the start: 21 parts, among them J11 Con_01x02_2.5mm, Q601 BSS138

Commit message: Add a connector next to the SHUTDOWN switch. Add 3D file for relay.
Parts:
- R101: now left out of the parts list
Changed lines of the file:
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@@
   )
   (symbol (lib_id "Device:R") (at 119.38 137.16 90) (mirror x) (unit 1)
-    (in_bom yes) (on_board yes) (dnp yes)
+    (in_bom no) (on_board yes) (dnp yes)
     (property "Reference" "R101" (at 120.65 132.08 90)
       (effects (font (size 1.27 1.27)))
