File: elec/Control Board/Control_1v2/Fan controller.kicad_sch (KiCad schematic)
At the start: 37 parts, among them J10 Conn_01x05, J11 Conn_01x04, J12 Conn_01x07, J20 Conn_01x04_KK-254_0470531000, J6 DB25_Female_MountingHoles, J9 Conn_01x04, Q2 NCE01P30K, Q601 BSS138

Commit message: PCB V1.2. Add test points of many colors.
Parts:
- TP103: Cost NA -> 0.0696; Distributor 1 (none) -> JLCPCB; Distributor 1 PN (none) -> C5277086; MPN (none) -> RH-5000; Manufacturer (none) -> ronghe
- TP103: Cost NA -> 0.1865; Distributor 1 (none) -> JLCPCB; Distributor 1 PN (none) -> C7589090; MPN (none) -> RH-5121; Manufacturer (none) -> ronghe
Changed lines of the file:
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@@
       (effects (font (size 1.27 1.27)) hide)
     )
-    (property "Cost" "NA" (at 137.16 57.15 0)
+    (property "Cost" "0.0696" (at 137.16 57.15 0)
+      (effects (font (size 1.27 1.27)) hide)
+    )
+    (property "Description" "Test Points/Test Rings ROHS red" (at 137.16 57.15 0)
+      (effects (font (size 1.27 1.27)) hide)
+    )
+    (property "Distributor 1" "JLCPCB" (at 137.16 57.15 0)
+      (effects (font (size 1.27 1.27)) hide)
+    )
+    (property "Distributor 1 PN" "C5277086" (at 137.16 57.15 0)
+      (effects (font (size 1.27 1.27)) hide)
+    )
+    (property "MPN" "RH-5000 " (at 137.16 57.15 0)
+      (effects (font (size 1.27 1.27)) hide)
+    )
+    (property "Manufacturer" "ronghe " (at 137.16 57.15 0)
       (effects (font (size 1.27 1.27)) hide)
     )
@@
       (effects (font (size 1.27 1.27)) hide)
     )
-    (property "Cost" "NA" (at 101.6 68.58 0)
-      (effects (font (size 1.27 1.27)) hide)
-    )
+    (property "Cost" "0.1865" (at 101.6 68.58 0)
+      (effects (font (size 1.27 1.27)) hide)
+    )
+    (property "Description" "Test Points/Test Rings ROHS green" (at 101.6 68.58 0)
+      (effects (font (size 1.27 1.27)) hide)
+    )
+    (property "Distributor 1 PN" "C7589090" (at 101.6 68.58 0)
+      (effects (font (size 1.27 1.27)) hide)
+    )
+    (property "Distributor 1" "JLCPCB" (at 101.6 68.58 0)
+      (effects (font (size 1.27 1.27)) hide)
+    )
+    (property "MPN" "RH-5121" (at 101.6 68.58 0)
+      (effects (font (size 1.27 1.27)) hide)
+    )
+    (property "Manufacturer" "ronghe " (at 101.6 68.58 0)
+      (effects (font (size 1.27 1.27)) hide)
+    )

Commit message: Set J20 for JLCPCB part number in Distirbutor 1.
Parts:
- J20: Distributor 1 Digikey -> JLCPCB; Distributor 1 PN WM4330-ND -> C3025061; Distributor 2 JLCPCB -> Digikey; Distributor 2 PN C3025061 -> WM4330-ND
Changed lines of the file:
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@@
       (effects (font (size 1.27 1.27)) hide)
     )
-    (property "Distributor 1" "Digikey" (at 222.25 81.28 0)
+    (property "Distributor 1" "JLCPCB" (at 222.25 81.28 0)
       (effects (font (size 1.27 1.27)) hide)
     )
-    (property "Distributor 1 PN" "WM4330-ND" (at 222.25 81.28 0)
+    (property "Distributor 1 PN" "C3025061" (at 222.25 81.28 0)
       (effects (font (size 1.27 1.27)) hide)
     )
-    (property "Distributor 2" "JLCPCB" (at 222.25 81.28 0)
+    (property "Distributor 2" "Digikey" (at 222.25 81.28 0)
       (effects (font (size 1.27 1.27)) hide)
     )
-    (property "Distributor 2 PN" "C3025061" (at 222.25 81.28 0)
+    (property "Distributor 2 PN" "WM4330-ND" (at 222.25 81.28 0)
       (effects (font (size 1.27 1.27)) hide)
     )
